File: Rough_Draft_Schematic.sch (EAGLE design)
At the start: 13 parts, among them IC1 ESP-12E/F, Q1 2N2102, SW1 CT10-XXXX-A2

Commit message: Add files via upload
Parts:
- removed SW1: CT10-XXXX-A2, switch-coto:CT10-XXXX-A2
- added S1: (no value), switch-omron:10-XX
Connections:
- net GND: now also S1.P1; no longer SW1.1
- net N$8: now also S1.S1; no longer SW1.2
Other:
- note added: "NOTES ************* 1. We have updated VCC. 2. We have tidied a few things up. QUESTIONS *************** 1. Does the Moisture Sensor need to be connected to the clock? 2. What kind of voltage regulator will we use?"
- note removed: "NOTES ***************** 1. We need to create EagleCAD parts for the sensors and actuator. Currently, we are using pin headers. 2. We need to possibly add a voltage regulator. 3. The base resistor of the motor-driving transistor might need to be tweaked for minimal power dissipation. 4. Additional circuitry (LED's, etc.) will be added if time permits."
- note removed: "QUESTIONS ******************** 1. How do we represent a pump (motor) in EagleCAD? 2. Should there be references in the schematic to mechanical devices (water resevoir, soil, etc.)?"
Changed lines of the file:
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@@
 <parts>
 <part name="IC1" library="esp-12e-f" deviceset="ESP-12E/F" device=""/>
-<part name="VDD1" library="supply1" library_urn="urn:adsk.eagle:library:371" deviceset="VDD" device="" value="5V"/>
+<part name="VDD1" library="supply1" library_urn="urn:adsk.eagle:library:371" deviceset="VDD" device="" value="7.4"/>
 <part name="JP3" library="pinhead" library_urn="urn:adsk.eagle:library:325" deviceset="PINHD-1X3" device="" package3d_urn="urn:adsk.eagle:package:22458/2"/>
 <part name="SUPPLY1" library="supply2" library_urn="urn:adsk.eagle:library:372" deviceset="GND" device=""/>
@@
 <part name="R5" library="rcl" library_urn="urn:adsk.eagle:library:334" deviceset="R-US_" device="0204/2V" package3d_urn="urn:adsk.eagle:package:23495/1" value="10k"/>
 <part name="R6" library="rcl" library_urn="urn:adsk.eagle:library:334" deviceset="R-US_" device="0204/2V" package3d_urn="urn:adsk.eagle:package:23495/1" value="10k"/>
-<part name="SW1" library="switch-coto" library_urn="urn:adsk.eagle:library:374" deviceset="CT10-XXXX-" device="A2" package3d_urn="urn:adsk.eagle:package:27090/1"/>
 <part name="JP5" library="pinhead" library_urn="urn:adsk.eagle:library:325" deviceset="PINHD-1X4" device="" package3d_urn="urn:adsk.eagle:package:22407/2"/>
 <part name="Q1" library="transistor-npn" library_urn="urn:adsk.eagle:library:398" deviceset="2N2102" device="" package3d_urn="urn:adsk.eagle:package:28729/1"/>
 <part name="R1" library="rcl" library_urn="urn:adsk.eagle:library:334" deviceset="R-US_" device="0204/2V" package3d_urn="urn:adsk.eagle:package:23495/1" value="1k"/>
+<part name="S1" library="switch-omron" library_urn="urn:adsk.eagle:library:377" deviceset="10-XX" device="" package3d_urn="urn:adsk.eagle:package:27496/1"/>
 </parts>
 <sheets>
@@
 <text x="162.56" y="99.06" size="1.778" layer="91">Water Pump</text>
 <text x="154.94" y="50.8" size="1.778" layer="91">Motor Drive Transistor</text>
-<text x="185.42" y="162.56" size="1.778" layer="91">NOTES
-*****************
-1. We need to create EagleCAD parts for the sensors and actuator. Currently, we are using pin headers.
-2. We need to possibly add a voltage regulator.
-3. The base resistor of the motor-driving transistor might need to be tweaked for minimal power dissipation.
-4. Additional circuitry (LED's, etc.) will be added if time permits.</text>
-<text x="185.42" y="124.46" size="1.778" layer="91">QUESTIONS
-********************
-1. How do we represent a pump (motor) in EagleCAD?
-2. Should there be references in the schematic to mechanical devices (water resevoir, soil, etc.)?</text>
+<text x="218.44" y="127" size="1.778" layer="91">NOTES
+*************
+1. We have updated VCC.
+2. We have tidied a few things up.
+QUESTIONS
+***************
+1. Does the Moisture Sensor need to be connected to the clock?
+2. What kind of voltage regulator will we use?</text>
 </plain>
 <instances>
@@
 <attribute name="VALUE" x="99.822" y="85.09" size="1.778" layer="96" rot="R90"/>
 </instance>
-<instance part="SW1" gate="G$1" x="114.3" y="60.96" smashed="yes" rot="R90">
-<attribute name="NAME" x="111.76" y="57.15" size="1.778" layer="95" rot="R90"/>
-<attribute name="VALUE" x="118.11" y="57.15" size="1.778" layer="96" rot="R90"/>
-</instance>
 <instance part="JP5" gate="A" x="43.18" y="-15.24" smashed="yes" rot="R90">
 <attribute name="VALUE" x="50.8" y="-21.59" size="1.778" layer="96" rot="R90"/>
 </instance>
 <instance part="Q1" gate="G$1" x="152.4" y="50.8" smashed="yes">
-<attribute name="NAME" x="142.24" y="58.42" size="1.778" layer="95"/>
-<attribute name="VALUE" x="142.24" y="55.88" size="1.778" layer="96"/>
+<attribute name="NAME" x="149.86" y="55.88" size="1.778" layer="95"/>
+<attribute name="VALUE" x="144.78" y="45.72" size="1.778" layer="96"/>
 </instance>
 <instance part="R1" gate="G$1" x="137.16" y="50.8" smashed="yes" rot="R180">
-<attribute name="NAME" x="140.97" y="49.3014" size="1.778" layer="95" rot="R180"/>
-<attribute name="VALUE" x="140.97" y="54.102" size="1.778" layer="96" rot="R180"/>
+<attribute name="NAME" x="138.43" y="49.3014" size="1.778" layer="95" rot="R180"/>
+<attribute name="VALUE" x="138.43" y="54.102" size="1.778" layer="96" rot="R180"/>
+</instance>
+<instance part="S1" gate="1" x="111.76" y="60.96" smashed="yes">
+<attribute name="NAME" x="115.57" y="58.42" size="1.778" layer="95" rot="R90"/>
+<attribute name="VALUE" x="107.95" y="64.135" size="1.778" layer="96" rot="R90"/>
 </instance>
 </instances>
@@
 <wire x1="96.52" y1="0" x2="96.52" y2="27.94" width="0.1524" layer="91"/>
 <wire x1="109.22" y1="0" x2="109.22" y2="-20.32" width="0.1524" layer="91"/>
-<pinref part="SW1" gate="G$1" pin="1"/>
 <wire x1="114.3" y1="55.88" x2="114.3" y2="-20.32" width="0.1524" layer="91"/>
 <junction x="114.3" y="-20.32"/>
@@
 <wire x1="154.94" y1="-20.32" x2="119.38" y2="-20.32" width="0.1524" layer="91"/>
 <junction x="119.38" y="-20.32"/>
+<pinref part="S1" gate="1" pin="P1"/>
 </segment>
 </net>
@@
 <wire x1="114.3" y1="78.74" x2="114.3" y2="66.04" width="0.1524" layer="91"/>
 <junction x="96.52" y="78.74"/>
-<pinref part="SW1" gate="G$1" pin="2"/>
-</segment>
-</net>
+<pinref part="S1" gate="1" pin="S1"/>
+</segment>
+</net>
